File: hardware/lightcube.kicad_pcb (KiCad board)
At the start: 2 copper layers, 12 parts, among them P1 IN, P2 OUT, P3 LED, Q1 MOSFET_N, Q2 MOSFET_N, Q3 MOSFET_N, U1 ATTINY25-SS

Commit message: Add programming pads
Signed-off-by: Paul Brook <paul@nowt.org>
Parts:
- added P4: PROG, prog_pads, B.Cu at (38.1, 41.9)
- P3: footprint SIL-4 -> SIL-4-ELL
- moved LOGO_SMALL 0.80 mm to (29.2, 44.5)
- moved Q2 0.63 mm to (36.8, 34.3)
Connections:
- P3 pad 2: /Rl -> /Gl
- P3 pad 3: /Gl -> /Rl
- Q1 pad D: /Rl -> /Gl
- Q1 pad G: /R -> /G
- Q2 pad D: /Gl -> /Rl
- Q2 pad G: /G -> /R
- U1 pad 1: (no net) -> /RESET
- U1 pad 3: /G -> /R
- U1 pad 5: /R -> /G
Routing:
- net /DI: track 10.6 -> 15.5 mm, vias 0 -> 1
- net /R: track 4.64 -> 9.55 mm, vias 0 -> 1
- net /RESET: track 0.00 -> 4.02 mm, vias 0 -> 1
- net /B: track 9.72 -> 12.4 mm, vias 0 -> 1
- net /G: track 10.2 -> 7.83 mm
- net /5v: track 10.8 -> 11.6 mm
Other:
- board text added: "A"
- board text added: "B"
- board text added: "G"
- board text added: "R"
